File: apps/hardware/kicad/studio/pcb-a/pcb-a.kicad_pcb (KiCad board)
At the start: 2 copper layers, 0 parts

Commit message: feat(hardware): PCB-A ubicada y ruteada (DRC limpio contra reglas de JLCPCB)
- tools/place_pcb_a.py: 5 EC11 bajo sus agujeros, pots IN/VOL en los brazos (15, 96) y (165, 96),
  6 separadores M3 (los 4 que pasan por PCB-K + uno por brazo), capacitores de 10 nF junto a cada pin.
- J2 (IDC 2×15) en la cara inferior hacia la portadora; J1 (JST-SH) ~40 mm al frente del J1 de PCB-K
  y mirándolo, para un cable de 50 mm en diagonal dentro del hueco de 7 mm.
- Ruteo con Freerouting (tools/route_board.py): zonas de exclusión sobre los agujeros sin cobre (el
  router no los ve) y limpieza de tramos sueltos; GND por planos con costura.
- Pads de GND de los conectores con unión sólida al plano (evita alivios térmicos de un solo radio);
  aplicado también a PCB-K.
- DRC con paridad de esquemático en las dos placas: 0 violaciones, 0 pads sin conectar.
- PROVISIONAL: brazos de los pots según un módulo Freenove de ~121 mm (medir antes del pedido).

Co-Authored-By: Claude Opus 5.5 <noreply@anthropic.com>
Parts:
- added C1: 10nF, Capacitor_SMD:C_0603_1608Metric, B.Cu at (71.0, 135.5)
- added C10: 10nF, Capacitor_SMD:C_0603_1608Metric, B.Cu at (71.0, 165.5)
- added C11: 10nF, Capacitor_SMD:C_0603_1608Metric, B.Cu at (71.0, 170.5)
- added C12: 10nF, Capacitor_SMD:C_0603_1608Metric, B.Cu at (93.0, 170.5)
- added C13: 10nF, Capacitor_SMD:C_0603_1608Metric, B.Cu at (187.0, 165.5)
- added C14: 10nF, Capacitor_SMD:C_0603_1608Metric, B.Cu at (187.0, 170.5)
- added C15: 10nF, Capacitor_SMD:C_0603_1608Metric, B.Cu at (209.0, 170.5)
- added C16: 100nF, Capacitor_SMD:C_0603_1608Metric, B.Cu at (65.0, 108.3)
- added C17: 100nF, Capacitor_SMD:C_0603_1608Metric, B.Cu at (215.0, 108.3)
- added C18: 10uF, Capacitor_SMD:C_0805_2012Metric, B.Cu at (145.2, 135.5)
- added C2: 10nF, Capacitor_SMD:C_0603_1608Metric, B.Cu at (71.0, 140.5)
- added C3: 10nF, Capacitor_SMD:C_0603_1608Metric, B.Cu at (93.0, 140.5)
- added C4: 10nF, Capacitor_SMD:C_0603_1608Metric, B.Cu at (187.0, 135.5)
- added C5: 10nF, Capacitor_SMD:C_0603_1608Metric, B.Cu at (187.0, 140.5)
- added C6: 10nF, Capacitor_SMD:C_0603_1608Metric, B.Cu at (209.0, 140.5)
- added C7: 10nF, Capacitor_SMD:C_0603_1608Metric, B.Cu at (129.0, 165.5)
- added C8: 10nF, Capacitor_SMD:C_0603_1608Metric, B.Cu at (129.0, 170.5)
- added C9: 10nF, Capacitor_SMD:C_0603_1608Metric, B.Cu at (151.0, 170.5)
- added ENC1: EC11 ENC L, Rotary_Encoder:RotaryEncoder_Alps_EC11E-Switch_Vertical_H20mm_MountingHoles, F.Cu at (74.5, 135.5)
- added ENC2: EC11 ENC R, Rotary_Encoder:RotaryEncoder_Alps_EC11E-Switch_Vertical_H20mm_MountingHoles, F.Cu at (190.5, 135.5)
- added ENC3: EC11 NAV, Rotary_Encoder:RotaryEncoder_Alps_EC11E-Switch_Vertical_H20mm_MountingHoles, F.Cu at (132.5, 165.5)
- added ENC4: EC11 P1, Rotary_Encoder:RotaryEncoder_Alps_EC11E-Switch_Vertical_H20mm_MountingHoles, F.Cu at (74.5, 165.5)
- added ENC5: EC11 P2, Rotary_Encoder:RotaryEncoder_Alps_EC11E-Switch_Vertical_H20mm_MountingHoles, F.Cu at (190.5, 165.5)
- added J1: A PCB-K (JST-SH 10), Connector_JST:JST_SH_SM10B-SRSS-TB_1x10-1MP_P1.00mm_Horizontal, F.Cu at (100.0, 148.0)
- added J2: A portadora (IDC 2x15), Connector_IDC:IDC-Header_2x15_P2.54mm_Vertical, B.Cu at (180.8, 129.3)
- added RV1: B10K IN, Potentiometer_THT:Potentiometer_Alpha_RD901F-40-00D_Single_Vertical, F.Cu at (62.5, 111.5)
- added RV2: B10K VOL, Potentiometer_THT:Potentiometer_Alpha_RD901F-40-00D_Single_Vertical, F.Cu at (212.5, 111.5)
Routing:
- net /+3V3: track 0.00 -> 187.5 mm, vias 0 -> 3
- net /P1_A: track 0.00 -> 124.3 mm, vias 0 -> 1
- net /P1_B: track 0.00 -> 111.7 mm, vias 0 -> 1
- net /ENCL_B: track 0.00 -> 104.5 mm, vias 0 -> 1
- net /+5V: track 0.00 -> 102.9 mm, vias 0 -> 2
- net /B2: track 0.00 -> 100.5 mm, vias 0 -> 2
- net /ENCL_A: track 0.00 -> 99.4 mm
- net /POT_IN: track 0.00 -> 99.3 mm
- net /P1_SW: track 0.00 -> 95.9 mm, vias 0 -> 1
- net /B4: track 0.00 -> 93.6 mm, vias 0 -> 2
- net /P2_SW: track 0.00 -> 92.7 mm, vias 0 -> 1
- net /B1: track 0.00 -> 92.2 mm, vias 0 -> 2
- net /LED_DIN: track 0.00 -> 88.2 mm, vias 0 -> 1
- net /B5: track 0.00 -> 83.4 mm, vias 0 -> 1
- net /POT_VOL: track 0.00 -> 82.4 mm, vias 0 -> 1
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- added copper zone on B.Cu, net /GND
- added copper zone on F.Cu, net /GND
Other:
- board outline added: 168 x 88 mm

Commit message: feat(hardware): enclosure +15 mm, PCB-A de una cara y ubicación de la portadora
Enclosure (design/README.md, theory/02 §3 y §4.3–4.5), medido el módulo Freenove con la Pi:
- Cuña de 43/78 mm (+15 mm parejo, 12°): la portadora entra bajo la Pi con margen y hay más aire.
- Pantalla corrida 2.5 mm hacia atrás (centro y 114.9): el vidrio (120.8 × 76 × 7.6 mm) ya no se monta
  sobre PCB-K; ranuras de aire en y 155–165.
- Pi atornillada detrás de la Freenove, puertos hacia la derecha (adentro): se elimina la tapa de servicio.
- Jacks en una hilera baja soldados a la portadora (1/4" NRJ3HF-1); USB y palanca PAD de panel arriba.
  La placa trasera vertical se descartó antes de commit.

PCB-A: todos los SMD en la cara superior (ensamble Economic de una cara); vía propia para los GND del
JST; re-ruteada. DRC 0/0.

Portadora: tools/place_portadora.py (97 × 100 mm, jacks contra la pared, shield y entrada analógica al
medio, Teensy y alimentación adelante, J5/J6 al frente). DRC con paridad: 0 violaciones; falta rutear.
Herramientas: costura de GND que respeta agujeros e islas, route_board sin duplicar lo bloqueado,
sync_fp_fields con redes "unconnected" y atributos de BOM, trim_silk_outside.py.

Co-Authored-By: Claude Opus 5.5 <noreply@anthropic.com>
Parts:
- C1, C10, C11, C12, C13, C14, C15, C16, C17, C18, C2, C3, C4, C5, C6, C7, C8, C9: moved to F.Cu
- moved C16 8.63 mm to (59.0, 114.5), turned to 0 degrees
- moved C17 8.63 mm to (209.0, 114.5), turned to 0 degrees
Routing:
- net /POT_VOL: track 82.4 -> 125.8 mm, vias 1 -> 3
- net /P1_A: track 124.3 -> 111.4 mm
- net /B1: track 92.2 -> 104.8 mm
- net /P2_B: track 78.7 -> 67.0 mm, vias 1 -> 0
- net /B2: track 100.5 -> 90.3 mm, vias 2 -> 1
- net /B6: track 77.8 -> 87.5 mm, vias 1 -> 2
- net /P1_B: track 111.7 -> 120.3 mm
- net /P2_A: track 68.9 -> 76.8 mm
- net /NAV_A: track 50.4 -> 58.2 mm
- net /NAV_B: track 60.8 -> 67.7 mm
- net /P1_SW: track 95.9 -> 102.4 mm
- net /+5V: track 102.9 -> 96.9 mm, vias 2 -> 1
- net /POT_IN: track 99.3 -> 105.0 mm
- net /B4: track 93.6 -> 89.0 mm
- net /ENCL_B: track 104.5 -> 100.1 mm, vias 1 -> 0
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
Commit message: feat(hardware): portadora ruteada (DRC limpio) y pinout del IDC reordenado
- Portadora: ruteo completo, DRC con paridad de esquemático 0/0/0 contra reglas de JLCPCB.
  +5V de F1 a la Pi en ~40 mm con una vía; sin paralelos audio↔digital a <1 mm.
- IDC 2×15 (PCB-A J2 ↔ portadora J5): pines ordenados por la X del pin de la Teensy al que van,
  para que el bus salga del conector sin cruces. Ambos esquemáticos re-etiquetados (ERC limpio),
  PCB-A re-ruteada (DRC 0/0/0). Tablas y razón en theory/02 §6.2.
- Herramientas: grid_route (Dijkstra en grilla 0.1 mm, 2 capas), finish_routing (rip-up and
  reroute de lo que deja Freerouting), clean_vias, add_gnd_escapes, fix_portadora_gnd,
  set_idc_pinout y build_portadora.sh (pipeline completo reproducible).

Co-Authored-By: Claude Opus 5.5 <noreply@anthropic.com>
Connections:
- J2 pad 11: /B5 -> /NAV_B
- J2 pad 12: /B6 -> /NAV_A
- J2 pad 13: /ENCL_A -> /P2_SW
- J2 pad 14: /ENCL_B -> /ENCR_SW
- J2 pad 15: /ENCL_SW -> /ENCL_A
- J2 pad 16: /ENCR_A -> /ENCR_B
- J2 pad 17: /ENCR_B -> /ENCL_B
- J2 pad 18: /ENCR_SW -> /ENCR_A
- J2 pad 19: /NAV_A -> /ENCL_SW
- J2 pad 20: /NAV_B -> /B6
- J2 pad 21: /NAV_SW -> /POT_IN
- J2 pad 22: /P1_A -> /B5
- J2 pad 23: /P1_B -> /NAV_SW
- J2 pad 24: /P1_SW -> /P2_B
- J2 pad 25: /P2_A -> /P1_A
- J2 pad 26: /P2_B -> /LED_DIN
- J2 pad 27: /P2_SW -> /P2_A
- J2 pad 28: /POT_IN -> /P1_B
- J2 pad 29: /POT_VOL -> /P1_SW
- J2 pad 5: /LED_DIN -> /B1
- J2 pad 7: /B1 -> /B2
- J2 pad 8: /B2 -> /POT_VOL
Routing:
- net /POT_VOL: track 125.8 -> 57.1 mm, vias 3 -> 2
- net /P2_SW: track 91.9 -> 62.2 mm, vias 1 -> 0
- net /P1_SW: track 102.4 -> 83.0 mm
- net /LED_DIN: track 86.7 -> 70.8 mm
- net /NAV_B: track 67.7 -> 82.0 mm, vias 0 -> 2
- net /P1_B: track 120.3 -> 106.8 mm
- net /B6: track 87.5 -> 74.7 mm, vias 2 -> 1
- net /B1: track 104.8 -> 92.9 mm, vias 2 -> 1
- net /B4: track 89.0 -> 79.7 mm, vias 2 -> 1
- net /NAV_A: track 58.2 -> 67.6 mm, vias 1 -> 0
- net /P1_A: track 111.4 -> 102.8 mm
- net /POT_IN: track 105.0 -> 112.7 mm
- net /ENCL_A: track 102.9 -> 95.4 mm, vias 1 -> 0
- net /P2_B: track 67.0 -> 61.0 mm
- net /+3V3: track 184.9 -> 178.9 mm, vias 0 -> 1
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
Commit message: feat(studio): prototipo económico de 2 placas, enclosure validado en FreeCAD y conectores de chasis
Placas (ADR-004 rev. 3, theory/02 §10F):
- Sin PCB-K ni LEDs montados: los Choc se cablean a J1 de PCB-A, que pasa de JST-SH a header 1×10 acodado
  con el mismo pinout (+5V y LED_DIN libres). PCB-A re-ruteada (build_pcb_a.sh), DRC con paridad 0/0/0.
- Portadora con ensamble solo de SMD; PCB-A solo PCB. export_fab.py genera solo esas dos.
- Todos los conectores traseros de chasis, cableados a los pads de los footprints de jacks (§10H).

Enclosure (apps/design/3d-models/studio, theory/02 §10E–10H):
- Modelo FreeCAD con las placas de KiCad: caja 48/83 a 12°, portadora corrida +16 mm en X para librar el
  GPIO de la Pi con el shield sobre headers.
- Pantalla sujeta con dos barras de PETG a 4 espárragos PEM; aluminio fijado con 6 M3 avellanados.
- Pared trasera en una sola fila (z 22), HOST en USB-A; separadores de la portadora y patas.
- Anillo WS2812 de NAV bajo un difusor Ø44 y soportes impresos para APA102 bajo cada Choc.
- Archivos: cuerpo-petg.stl, barras, soportes de tecla, panel-aluminio.dxf (3 capas), difusor-nav.dxf.

Co-Authored-By: Claude Opus 5.5 <noreply@anthropic.com>
Parts:
- J1: value A PCB-K (JST-SH 10) -> A Choc + LEDs (1x10 acodado); footprint Connector_JST:JST_SH_SM10B-SRSS-TB_1x10-1MP_P1.00mm_Horizontal -> Connector_PinHeader_2.54mm:PinHeader_1x10_P2.54mm_Horizontal
- moved J1 9.43 mm to (100.0, 138.6), turned to 0 degrees
Routing:
- net /P1_A: track 102.8 -> 128.0 mm
- net /B5: track 80.0 -> 95.4 mm
- net /GND: track 3.80 -> 18.1 mm, vias 231 -> 223
- net /NAV_B: track 82.0 -> 69.5 mm, vias 2 -> 1
- net /B6: track 74.7 -> 65.6 mm
- net /P1_SW: track 83.0 -> 91.7 mm
- net /LED_DIN: track 70.8 -> 77.3 mm
- net /POT_VOL: track 57.1 -> 52.0 mm
- net /B1: track 92.9 -> 89.0 mm, vias 1 -> 0
- net /B4: track 79.7 -> 76.1 mm, vias 1 -> 0
- net /ENCR_SW: track 52.9 -> 49.4 mm, vias 1 -> 0
- net /+3V3: track 178.9 -> 175.5 mm, vias 1 -> 0
- net /B3: track 80.0 -> 76.6 mm, vias 1 -> 0
- net /P1_B: track 106.8 -> 109.3 mm
- net /ENCR_B: track 38.5 -> 36.9 mm
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